Commit message: updated map corrected joint frame

File: whereAmI/src/my_robot/urdf/my_robot.xacro (robot description, xacro)
@@ -166,5 +166,5 @@
   </gazebo>
   <joint type="fixed" name="hokuyo_joint">
-    <origin xyz="0.15 0 0" rpy="-0.05 0 0"/>
+    <origin xyz="0.15 0 0.25" rpy="-0.05 0 0"/>
     <child link="hokuyo"/>
     <parent link="chassis"/>
